Commit message: Fixed warnings with xacro tags

File: rb_theron_description/robots/rb_theron.urdf.xacro (robot description, xacro)
@@ -9,11 +9,11 @@
 	<xacro:include filename="$(find rb_theron_description)/robots/rb_theron_base.urdf.xacro" />
 	<!-- Import wheels -->
-	<xacro:include filename="$(find rb_theron_description)/urdf/wheels/rubber_wheel_150.urdf.xacro" />
+	<!--xacro:include filename="$(find rb_theron_description)/urdf/wheels/rubber_wheel_150.urdf.xacro" /-->
 	<!-- Import casters -->
-	<xacro:include filename="$(find rb_theron_description)/urdf/wheels/castor.urdf.xacro" />
+	<!--xacro:include filename="$(find rb_theron_description)/urdf/wheels/castor.urdf.xacro" /-->
 	<!-- Import all available sensors -->
-	<xacro:include filename="$(find robotnik_sensors)/urdf/all_sensors.urdf.xacro" />
+	<!--xacro:include filename="$(find robotnik_sensors)/urdf/all_sensors.urdf.xacro" /-->
 	<!-- Import Gazebo Stuff -->
-	<xacro:include filename="$(find rb_theron_description)/urdf/common.gazebo.xacro" />
+	<!--xacro:include filename="$(find rb_theron_description)/urdf/common.gazebo.xacro" /-->
 	<!-- ***************** -->
 	<!-- Global parameters -->
@@ -34,9 +34,9 @@
 	<xacro:rb_theron_base prefix="$(arg prefix)" hq="${hq}" />
 	<!-- Gazebo ros control pluggins -->
-	<xacro:ros_control/>
-	<xacro:gazebo_colors prefix="$(arg prefix)"/>
+	<!--xacro:ros_control/-->
+	<!--xacro:gazebo_colors prefix="$(arg prefix)"/-->
   <!-- SENSORS -->
   <!-- TODO: Moved 0.01 in x, otherwise the camera is still inside the robot -->
-	<xacro:sensor_orbbec_astra prefix="$(arg prefix)front_rgbd_camera" parent="$(arg prefix)base_link" prefix_topic="front_rgbd_camera">
+	<!--xacro:sensor_orbbec_astra prefix="$(arg prefix)front_rgbd_camera" parent="$(arg prefix)base_link" prefix_topic="front_rgbd_camera">
 		<origin xyz="0.3305 0.0 0.1898" rpy="0 0 0"/>
 	</xacro:sensor_orbbec_astra>
@@ -46,4 +46,4 @@
 	<xacro:sensor_sick_nanoscan3 prefix="$(arg prefix)front_laser" parent="$(arg prefix)base_link" prefix_topic="front_laser" min_angle="-2.0507619" max_angle="2.0507619">
 		<origin xyz="0.250 0.0 0.1643" rpy="0 3.1416 3.1416"/>
-	</xacro:sensor_sick_nanoscan3>
+	</xacro:sensor_sick_nanoscan3-->
 </robot>

File: rb_theron_description/urdf/bases/theron_base.urdf.xacro (robot description, xacro)
@@ -2,9 +2,9 @@
 <robot name="rbogie_base"
   xmlns:xacro="http://www.ros.org/wiki/xacro">
-<macro name="box_inertia_robot" params="m x y z">
+<xacro:macro name="box_inertia" params="m x y z">
         <inertia  ixx="${m*(y*y+z*z)/12}" ixy = "0" ixz = "0"
                   iyy="${m*(x*x+z*z)/12}" iyz = "0"
                   izz="${m*(x*x+z*z)/12}" />
-</macro>
+</xacro:macro>
   <xacro:macro name="theron_base" params="prefix publish_bf hq">
     <!-- Robot mechanical and motor parameters -->
@@ -29,9 +29,5 @@
     <!-- BASE_LINK -->
     <link name="${prefix}base_link">
-      <inertial>
-      <mass value="45" />
-      <origin xyz="0.0 0.0 0.0" />
-      <xacro:solid_cuboid_inertia m="45" w="0.3275" h="0.2775" d="0.1525" />
-     </inertial>
+      <xacro:box_inertia m="45" x="0.3275" y="0.2775" z="0.1525" />
       <visual>
         <origin xyz="0 0 0" rpy="0 0 0" />

File: rb_theron_description/urdf/wheels/castor.urdf.xacro (robot description, xacro)
@@ -3,9 +3,9 @@
   <xacro:property name="M_PI" value="3.1415926535897931" />
   <!-- Caster support parameters -->
-  <property name="caster_support_mass" value="1.5" /> <!-- in kg-->
+  <xacro:property name="caster_support_mass" value="1.5" /> <!-- in kg-->
   <!-- Caster wheel parameters -->
-  <property name="caster_radius" value="0.050" />
-  <property name="caster_height" value="0.025" />
-  <property name="caster_mass" value="0.25" /> <!-- in kg-->
+  <xacro:property name="caster_radius" value="0.050" />
+  <xacro:property name="caster_height" value="0.025" />
+  <xacro:property name="caster_mass" value="0.25" /> <!-- in kg-->
   <!-- Caster wheel offset-->
   <xacro:property name="caster_wheel_offset_x" value="-0.033" />
@@ -23,5 +23,5 @@
       <parent link="${parent}"/>
       <child link="${prefix}support"/>
-      <insert_block name="origin" />
+      <xacro:insert_block name="origin" />
       <axis xyz="0 0 1" rpy="0 ${M_PI} 0" />
       <limit effort="100" velocity="100"/>
@@ -45,5 +45,5 @@
         <mass value="${caster_support_mass}" />
         <origin xyz="0 0 0" />
-        <cylinder_inertia  m="${caster_support_mass}" r="0.010" h="0.010" />  <!--Check these values -->
+        <xacro:cylinder_inertia  m="${caster_support_mass}" r="0.010" h="0.010" />  <!--Check these values -->
       </inertial>
     </link>
@@ -58,5 +58,5 @@
        <parent link="${parent}"/>
        <child link="${prefix}wheel"/>
-       <insert_block name="origin" />
+       <xacro:insert_block name="origin" />
        <axis xyz="0 1 0" rpy="0 0 0" />
        <limit effort="100" velocity="100"/>
@@ -96,5 +96,5 @@
         <mass value="${caster_mass}" />
         <origin xyz="0 0 0" />
-        <cylinder_inertia  m="${caster_mass}" r="${caster_radius}" h="${caster_height}" />
+        <xacro:cylinder_inertia  m="${caster_mass}" r="${caster_radius}" h="${caster_height}" />
       </inertial>
     </link>

Commit message: Fixed comentary error, ros2 control parser not allow /t ascci chars

File: rb_theron_description/robots/rb_theron.urdf.xacro (robot description, xacro)
@@ -16,4 +16,6 @@
 	<!-- Import Gazebo Stuff -->
 	<!--xacro:include filename="$(find rb_theron_description)/urdf/common.gazebo.xacro" /-->
+	<!-- Import differential base elements -->
+	<xacro:include filename="$(find rb_theron_description)/urdf/theron.ros2_control.xacro" />
 	<!-- ***************** -->
 	<!-- Global parameters -->
@@ -21,7 +23,7 @@
 	<xacro:property name="PI" value="3.1415926535897931"/>
 	<!-- Wheel parameters -->
-	<!--xacro:property name="wheel_offset_x" value="0" />
-	<xacro:property name="wheel_offset_y" value="0.2516" />
-	<xacro:property name="wheel_offset_z" value="0.0" /-->
+	<!--xacro:property name="wheel_offset_x" value="0" /-->
+	<!--xacro:property name="wheel_offset_y" value="0.2516" /-->
+	<!--xacro:property name="wheel_offset_z" value="0.0" /-->
 	<!-- Flag to select the high or low quality model -->
 	<xacro:property name="hq" value="true" />
@@ -33,17 +35,18 @@
 	<!-- base with wheels -->
 	<xacro:rb_theron_base prefix="$(arg prefix)" hq="${hq}" />
+	<xacro:example_ros2_control name="robotnik_demo_name" prefix="$(arg prefix)" />
 	<!-- Gazebo ros control pluggins -->
 	<!--xacro:ros_control/-->
 	<!--xacro:gazebo_colors prefix="$(arg prefix)"/-->
   <!-- SENSORS -->
-  <!-- TODO: Moved 0.01 in x, otherwise the camera is still inside the robot -->
-	<!--xacro:sensor_orbbec_astra prefix="$(arg prefix)front_rgbd_camera" parent="$(arg prefix)base_link" prefix_topic="front_rgbd_camera">
-		<origin xyz="0.3305 0.0 0.1898" rpy="0 0 0"/>
-	</xacro:sensor_orbbec_astra>
-	<xacro:sensor_imu_hector prefix="$(arg prefix)imu" parent="$(arg prefix)base_link">
-		<origin xyz="-0.1975 0.0 0.1598" rpy="0 0 0"/>
-	</xacro:sensor_imu_hector>
-	<xacro:sensor_sick_nanoscan3 prefix="$(arg prefix)front_laser" parent="$(arg prefix)base_link" prefix_topic="front_laser" min_angle="-2.0507619" max_angle="2.0507619">
-		<origin xyz="0.250 0.0 0.1643" rpy="0 3.1416 3.1416"/>
-	</xacro:sensor_sick_nanoscan3-->
+  <!-- TODO Moved 0.01 in x, otherwise the camera is still inside the robot -->
+	<!--xacro:sensor_orbbec_astra prefix="$(arg prefix)front_rgbd_camera" parent="$(arg prefix)base_link" prefix_topic="front_rgbd_camera"-->
+		<!--origin xyz="0.3305 0.0 0.1898" rpy="0 0 0"/-->
+	<!--/xacro:sensor_orbbec_astra-->
+	<!--xacro:sensor_imu_hector prefix="$(arg prefix)imu" parent="$(arg prefix)base_link"-->
+		<!--origin xyz="-0.1975 0.0 0.1598" rpy="0 0 0"/-->
+	<!--/xacro:sensor_imu_hector-->
+	<!--xacro:sensor_sick_nanoscan3 prefix="$(arg prefix)front_laser" parent="$(arg prefix)base_link" prefix_topic="front_laser" min_angle="-2.0507619" max_angle="2.0507619"-->
+		<!--origin xyz="0.250 0.0 0.1643" rpy="0 3.1416 3.1416"/-->
+	<!--/xacro:sensor_sick_nanoscan3-->
 </robot>

File: rb_theron_description/urdf/rocker/mcq_prototype_rocker.urdf.xacro (robot description, xacro)
@@ -100,20 +100,20 @@
 		<origin xyz="${caster_offset_x} ${caster_offset_y} ${caster_offset_z}" rpy="0 0 0"/>
 	</xacro:caster>
-    <!-- gazebo reference="${prefix}support">
-			<mu1 value="5.0"/>
-			<mu2 value="0.5"/>
-			<kp value="10000000.0" />
-			<kd value="1.0" />
-			<fdir1 value="1 0 0"/>
-      <turnGravityOff>false</turnGravityOff>
-    </gazebo>
-     <gazebo reference="${prefix}_wheel">
-			<mu1 value="5.0"/>
-			<mu2 value="0.5"/>
-			<kp value="10000000.0" />
-			<kd value="1.0" />
-			<fdir1 value="1 0 0"/>
-      <turnGravityOff>false</turnGravityOff>
-    </gazebo -->
+    <!-- gazebo reference="${prefix}support"-->
+			<!--mu1 value="5.0"/-->
+			<!--mu2 value="0.5"/-->
+			<!--kp value="10000000.0" /-->
+			<!--kd value="1.0" /-->
+			<!--fdir1 value="1 0 0"/-->
+      <!--turnGravityOff>false</turnGravityOff-->
+    <!--/gazebo-->
+     <!--gazebo reference="${prefix}_wheel"-->
+			<!--mu1 value="5.0"/-->
+			<!--mu2 value="0.5"/-->
+			<!--kp value="10000000.0" /-->
+			<!--kd value="1.0" /-->
+			<!--fdir1 value="1 0 0"/-->
+      <!--turnGravityOff>false</turnGravityOff-->
+    <!--/gazebo -->
  </xacro:macro>
 </robot>

File: rb_theron_description/urdf/wheels/castor.urdf.xacro (robot description, xacro)
@@ -36,10 +36,10 @@
           </geometry>
       </visual>
-      <!--collision>
-        <origin xyz="0 0 0" rpy="0 0 0" />
-          <geometry>
-	       <mesh filename="package://rb_theron_description/meshes/wheels/castor_wheel.dae" />
-          </geometry>
-      </collision-->
+      <!--collision-->
+        <!--origin xyz="0 0 0" rpy="0 0 0" /-->
+          <!--geometry-->
+	       <!--mesh filename="package://rb_theron_description/meshes/wheels/castor_wheel.dae" /-->
+          <!--/geometry-->
+      <!--/collision-->
       <inertial>
         <mass value="${caster_support_mass}" />
@@ -66,10 +66,10 @@
       <visual>
         <!-- HIGH RESOLUTION WHEELS -->
-     <!-- xacro:if value="${hq}">
-          <origin xyz="0 0 0" rpy="0 0 0" />
-          <geometry>
-		<mesh filename="package://rb_theron_description/meshes/wheels/mcq_prototype_castor_wheel.dae" />
-          </geometry>
-        </xacro:if -->
+     <!-- xacro:if value="${hq}"-->
+          <!--origin xyz="0 0 0" rpy="0 0 0" /-->
+          <!-- geometry-->
+		<!--mesh filename="package://rb_theron_description/meshes/wheels/mcq_prototype_castor_wheel.dae" /-->
+          <!--/geometry-->
+        <!--/xacro:if -->
        <!-- LOW RESOLUTION WHEELS -->
        <!-- xacro:unless value="${hq}" -->
@@ -120,12 +120,12 @@
       </actuator>
     </transmission>
-    <!-- gazebo reference="${prefix}support">
-			<mu1 value="5.0"/>
-			<mu2 value="0.5"/>
-			<kp value="10000000.0" />
-			<kd value="1.0" />
-			<fdir1 value="1 0 0"/>
-      <turnGravityOff>false</turnGravityOff>
-    </gazebo -->
+    <!-- gazebo reference="${prefix}support"-->
+			<!--mu1 value="5.0"/-->
+			<!--mu2 value="0.5"/-->
+			<!--kp value="10000000.0" /-->
+			<!--kd value="1.0" /-->
+			<!--fdir1 value="1 0 0"/-->
+      <!--turnGravityOff>false</turnGravityOff-->
+    <!--/gazebo -->
      <gazebo reference="${prefix}_wheel">
 			<mu1 value="100.0"/>

File: rb_theron_description/urdf/wheels/rubber_wheel.gazebo.xacro (robot description, xacro)
@@ -3,13 +3,13 @@
 	<xacro:macro name="rubber_wheel_gazebo" params="prefix">
 		<gazebo reference="${prefix}_wheel_link">
-			<!-- mu1 value="5.0"/>
-			<mu2 value="0.5"/>
-			<kp value="10000000.0" />
-			<kd value="1.0" />
-			<fdir1 value="1 0 0"/>
-			<material>Gazebo/Yellow</material>
-			<turnGravityOff>false</turnGravityOff -->
-			<!-- mu1 value="5.0"/>
-			<mu2 value="0.5"/ -->
+			<!--mu1 value="5.0"/-->
+			<!--mu2 value="0.5"/-->
+			<!--kp value="10000000.0" /-->
+			<!--kd value="1.0" /-->
+			<!--fdir1 value="1 0 0"/-->
+			<!--material>Gazebo/Yellow</material-->
+			<!--turnGravityOff>false</turnGravityOff -->
+			<!-- mu1 value="5.0"/-->
+			<!--mu2 value="0.5"/ -->
 			<mu1 value="100.0"/>
 			<mu2 value="100.0"/>
@@ -20,18 +20,18 @@
 			<material>Gazebo/Yellow</material>
 			<turnGravityOff>false</turnGravityOff>
-			<!--kp>500000.0</kp>
-			<kd>10.0</kd>
-			<mu1>10</mu1>
-			<mu2>10</mu2>
-			<fdir1>1 0 0</fdir1-->
+			<!--kp>500000.0</kp-->
+			<!--kd>10.0</kd-->
+			<!--mu1>10</mu1-->
+			<!--mu2>10</mu2-->
+			<!--fdir1>1 0 0</fdir1-->
 			<!--minDepth>0.001</minDepth-->
 			<!--material>Gazebo/Black</material-->
-			<!--mu1 value="10"/>
-			<mu2 value="5"/>
-			<kp value="500000.0" />
-			<kd value="10.0" />
-			<fdir1 value="1 0 0"/>
-			<material>Gazebo/Yellow</material>
-			<turnGravityOff>false</turnGravityOff-->
+			<!--mu1 value="10"/-->
+			<!--mu2 value="5"/-->
+			<!--kp value="500000.0" /-->
+			<!--kd value="10.0" /-->
+			<!--fdir1 value="1 0 0"/-->
+			<!--material>Gazebo/Yellow</material-->
+			<!--turnGravityOff>false</turnGravityOff-->
 		</gazebo>
 		<gazebo reference="${prefix}_wheel_tire_link">
@@ -39,16 +39,16 @@
 			<turnGravityOff>false</turnGravityOff>
 		</gazebo>
-		<!--gazebo reference="${name}_wheel_link">
-			<kp>500000.0</kp>
-			<kd>10.0</kd>
-			<mu1>10</mu1>
-			<mu2>10</mu2>
-			<fdir1>1 0 0</fdir1>
-			<maxVel>1.0</maxVel>
-			<minDepth>0.003</minDepth>
-			<material>Gazebo/Yellow</material>
-			<turnGravityOff>false</turnGravityOff>
-			<implicitSpringDamper>1</implicitSpringDamper>
-		</gazebo-->
+		<!--gazebo reference="${name}_wheel_link"-->
+			<!--kp>500000.0</kp-->
+			<!--kd>10.0</kd-->
+			<!--mu1>10</mu1-->
+			<!--mu2>10</mu2-->
+			<!--fdir1>1 0 0</fdir1-->
+			<!--maxVel>1.0</maxVel-->
+			<!--minDepth>0.003</minDepth-->
+			<!--material>Gazebo/Yellow</material-->
+			<!--turnGravityOff>false</turnGravityOff-->
+			<!--implicitSpringDamper>1</implicitSpringDamper-->
+		<!--/gazebo-->
 	</xacro:macro>
 </robot>

Commit message: Added hokuyo laser and changed joint type to fixed for caster wheels

File: rb_theron_description/robots/rb_theron.urdf.xacro (robot description, xacro)
@@ -13,5 +13,5 @@
 	<!--xacro:include filename="$(find rb_theron_description)/urdf/wheels/castor.urdf.xacro" /-->
 	<!-- Import all available sensors -->
-	<!--xacro:include filename="$(find robotnik_sensors)/urdf/all_sensors.urdf.xacro" /-->
+	<xacro:include filename="$(find robotnik_sensors)/urdf/all_sensors.urdf.xacro" />
 	<!-- Import Gazebo Stuff -->
 	<!--xacro:include filename="$(find rb_theron_description)/urdf/common.gazebo.xacro" /-->
@@ -44,4 +44,7 @@
 		<!--origin xyz="0.3305 0.0 0.1898" rpy="0 0 0"/-->
 	<!--/xacro:sensor_orbbec_astra-->
+	<xacro:sensor_hokuyo_ust10lx prefix="$(arg prefix)front_lidar" parent="$(arg prefix)base_link" prefix_topic="front_laser">
+		<origin xyz="0.3305 0.0 0.1898" rpy="${PI} 0 0"/>
+	</xacro:sensor_hokuyo_ust10lx>
 	<!--xacro:sensor_imu_hector prefix="$(arg prefix)imu" parent="$(arg prefix)base_link"-->
 		<!--origin xyz="-0.1975 0.0 0.1598" rpy="0 0 0"/-->

File: rb_theron_description/urdf/wheels/castor.urdf.xacro (robot description, xacro)
@@ -20,5 +20,5 @@
   <xacro:macro name="caster" params="prefix parent *origin hq">
   <!--CASTER SUPPORT -->
-  <joint name="${prefix}joint_support" type="continuous">
+  <joint name="${prefix}joint_support" type="fixed">
       <parent link="${parent}"/>
       <child link="${prefix}support"/>
@@ -55,5 +55,5 @@
  </xacro:macro>
  <xacro:macro name="caster_wheel" params="prefix parent *origin hq">
-     <joint name="${prefix}joint_wheel" type="continuous">
+     <joint name="${prefix}joint_wheel" type="fixed">
        <parent link="${parent}"/>
        <child link="${prefix}wheel"/>

Commit message: Removed robotnik_msgs dependency and create Dockerfile with instructions to generate image

File: rb_theron_description/robots/rb_theron.urdf.xacro (robot description, xacro)
@@ -13,9 +13,9 @@
 	<!--xacro:include filename="$(find rb_theron_description)/urdf/wheels/castor.urdf.xacro" /-->
 	<!-- Import all available sensors -->
-	<xacro:include filename="$(find robotnik_sensors)/urdf/all_sensors.urdf.xacro" />
+	<!--xacro:include filename="$(find robotnik_sensors)/urdf/all_sensors.urdf.xacro" /-->
 	<!-- Import Gazebo Stuff -->
 	<!--xacro:include filename="$(find rb_theron_description)/urdf/common.gazebo.xacro" /-->
 	<!-- Import differential base elements -->
-	<xacro:include filename="$(find rb_theron_description)/urdf/theron.ros2_control.xacro" />
+	<!--xacro:include filename="$(find rb_theron_description)/urdf/theron.ros2_control.xacro" /-->
 	<!-- ***************** -->
 	<!-- Global parameters -->
@@ -35,5 +35,5 @@
 	<!-- base with wheels -->
 	<xacro:rb_theron_base prefix="$(arg prefix)" hq="${hq}" />
-	<xacro:example_ros2_control name="robotnik_demo_name" prefix="$(arg prefix)" />
+	<!--xacro:example_ros2_control name="robotnik_demo_name" prefix="$(arg prefix)" log_level="info" /-->
 	<!-- Gazebo ros control pluggins -->
 	<!--xacro:ros_control/-->
@@ -44,7 +44,7 @@
 		<!--origin xyz="0.3305 0.0 0.1898" rpy="0 0 0"/-->
 	<!--/xacro:sensor_orbbec_astra-->
-	<xacro:sensor_hokuyo_ust10lx prefix="$(arg prefix)front_lidar" parent="$(arg prefix)base_link" prefix_topic="front_laser">
-		<origin xyz="0.3305 0.0 0.1898" rpy="${PI} 0 0"/>
-	</xacro:sensor_hokuyo_ust10lx>
+	<!--xacro:sensor_hokuyo_ust10lx prefix="$(arg prefix)front_lidar" parent="$(arg prefix)base_link" prefix_topic="front_laser"-->
+		<!--origin xyz="0.3305 0.0 0.1898" rpy="${PI} 0 0"/-->
+	<!--/xacro:sensor_hokuyo_ust10lx-->
 	<!--xacro:sensor_imu_hector prefix="$(arg prefix)imu" parent="$(arg prefix)base_link"-->
 		<!--origin xyz="-0.1975 0.0 0.1598" rpy="0 0 0"/-->

Commit message: Extract funcionality docker image out

File: rb_theron_description/robots/rb_theron.urdf.xacro (robot description, xacro)
@@ -8,22 +8,11 @@
 	<!-- Import differential base elements -->
 	<xacro:include filename="$(find rb_theron_description)/robots/rb_theron_base.urdf.xacro" />
-	<!-- Import wheels -->
-	<!--xacro:include filename="$(find rb_theron_description)/urdf/wheels/rubber_wheel_150.urdf.xacro" /-->
-	<!-- Import casters -->
-	<!--xacro:include filename="$(find rb_theron_description)/urdf/wheels/castor.urdf.xacro" /-->
 	<!-- Import all available sensors -->
-	<!--xacro:include filename="$(find robotnik_sensors)/urdf/all_sensors.urdf.xacro" /-->
-	<!-- Import Gazebo Stuff -->
-	<!--xacro:include filename="$(find rb_theron_description)/urdf/common.gazebo.xacro" /-->
-	<!-- Import differential base elements -->
-	<!--xacro:include filename="$(find rb_theron_description)/urdf/theron.ros2_control.xacro" /-->
+	<xacro:include filename="$(find robotnik_sensors)/urdf/all_sensors.urdf.xacro" />
 	<!-- ***************** -->
 	<!-- Global parameters -->
 	<!-- ***************** -->
-	<xacro:property name="PI" value="3.1415926535897931"/>
-	<!-- Wheel parameters -->
-	<!--xacro:property name="wheel_offset_x" value="0" /-->
-	<!--xacro:property name="wheel_offset_y" value="0.2516" /-->
-	<!--xacro:property name="wheel_offset_z" value="0.0" /-->
+	<!-- Prefix of robot frames -->
+	<xacro:arg name="prefix" default="robot_"/>
 	<!-- Flag to select the high or low quality model -->
 	<xacro:property name="hq" value="true" />
@@ -31,25 +20,6 @@
 	<!-- Robots Elements -->
 	<!-- *************** -->
-	<xacro:arg name="prefix" default="robot_"/>
 	<!-- Here we create the robot elements using the xacro:macros imported at the beggining of this file -->
 	<!-- base with wheels -->
 	<xacro:rb_theron_base prefix="$(arg prefix)" hq="${hq}" />
-	<!--xacro:example_ros2_control name="robotnik_demo_name" prefix="$(arg prefix)" log_level="info" /-->
-	<!-- Gazebo ros control pluggins -->
-	<!--xacro:ros_control/-->
-	<!--xacro:gazebo_colors prefix="$(arg prefix)"/-->
-  <!-- SENSORS -->
-  <!-- TODO Moved 0.01 in x, otherwise the camera is still inside the robot -->
-	<!--xacro:sensor_orbbec_astra prefix="$(arg prefix)front_rgbd_camera" parent="$(arg prefix)base_link" prefix_topic="front_rgbd_camera"-->
-		<!--origin xyz="0.3305 0.0 0.1898" rpy="0 0 0"/-->
-	<!--/xacro:sensor_orbbec_astra-->
-	<!--xacro:sensor_hokuyo_ust10lx prefix="$(arg prefix)front_lidar" parent="$(arg prefix)base_link" prefix_topic="front_laser"-->
-		<!--origin xyz="0.3305 0.0 0.1898" rpy="${PI} 0 0"/-->
-	<!--/xacro:sensor_hokuyo_ust10lx-->
-	<!--xacro:sensor_imu_hector prefix="$(arg prefix)imu" parent="$(arg prefix)base_link"-->
-		<!--origin xyz="-0.1975 0.0 0.1598" rpy="0 0 0"/-->
-	<!--/xacro:sensor_imu_hector-->
-	<!--xacro:sensor_sick_nanoscan3 prefix="$(arg prefix)front_laser" parent="$(arg prefix)base_link" prefix_topic="front_laser" min_angle="-2.0507619" max_angle="2.0507619"-->
-		<!--origin xyz="0.250 0.0 0.1643" rpy="0 3.1416 3.1416"/-->
-	<!--/xacro:sensor_sick_nanoscan3-->
 </robot>
